Commit message: added .dae meshes

File: descriptions/olympus_description/urdf/olympus.urdf (robot description, URDF)
Before this commit: robot olympus_description, 33 links, 32 joints
Links:
- link BackLeft_paw: geometry collision mesh filename=package://olympus_description/urdf/meshes/BackLeft_paw.dae; visual mesh filename=package://olympus_description/urdf/meshes/BackLeft_paw.dae
- link BackRight_paw: geometry collision mesh filename=package://olympus_description/urdf/meshes/BackRight_paw.dae; visual mesh filename=package://olympus_description/urdf/meshes/BackRight_paw.dae
- link Body: geometry collision mesh filename=package://olympus_description/urdf/meshes/Body.dae; visual mesh filename=package://olympus_description/urdf/meshes/Body.dae
- link FrontLeft_paw: geometry collision mesh filename=package://olympus_description/urdf/meshes/FrontLeft_paw.dae; visual mesh filename=package://olympus_description/urdf/meshes/FrontLeft_paw.dae
- link FrontRight_paw: geometry collision mesh filename=package://olympus_description/urdf/meshes/FrontRight_paw.dae; visual mesh filename=package://olympus_description/urdf/meshes/FrontRight_paw.dae

Commit message: Small corrcetion in placement of ankle joints

File: descriptions/olympus_description/urdf/olympus.urdf (robot description, URDF)
Before this commit: robot olympus_description, 33 links, 32 joints
Joints:
- joint BackLeft_ankle_inner_joint: origin xyz=0 0 -0.296 rpy=0 0 0 -> xyz=0 0 -0.29610 rpy=0 0 0
- joint BackLeft_ankle_outer_joint: origin xyz=0 0 -0.296 rpy=0 0 0 -> xyz=0 0 -0.29929 rpy=0 0 0
- joint BackRight_ankle_inner_joint: origin xyz=0 0 -0.296 rpy=0 0 0 -> xyz=0 0 -0.29610 rpy=0 0 0
- joint BackRight_ankle_outer_joint: origin xyz=0 0 -0.296 rpy=0 0 0 -> xyz=0 0 -0.29929 rpy=0 0 0
- joint FrontRight_ankle_inner_joint: origin xyz=0 0 -0.296 rpy=0 0 0 -> xyz=0 0 -0.29610 rpy=0 0 0
- joint FrontRight_ankle_outer_joint: origin xyz=0 0 -0.296 rpy=0 0 0 -> xyz=0 0 -0.29929 rpy=0 0 0
